Commit message: feat: both enemy and friendly tank have full collision, and inertia model, and both can be controlled via topic messages ps: yet you need to adjust the topic in the launchfile based on the robot you spawn to be able to control it

File: tank_robot/urdf/enemy_sim.urdf (robot description, URDF)
Before this commit: robot enemy_photo, 6 links, 5 joints
Joints:
- joint gun_joint: axis 0 1 0 -> 0 -1 0
